Commit message: today my .urdf.xacro file is updated date is 20/8/2025

File: src/dreamobot_description/urdf/dreambot.urdf.xacro (robot description, xacro)
@@ -15,4 +15,10 @@
       </geometry>
     </visual>
+    <collision>
+      <origin rpy="0 0 0" xyz="0 0 0"/>
+      <geometry>
+        <mesh filename="package://dreamobot_description/meshes/Circular_base.stl" scale="0.01 0.01 0.01"/>
+      </geometry>
+    </collision>
   </link>
   <!-- Fixed Joint: world -> base_link -->
