Commit message: Update at date 30/8/2025

File: install/dreamobot_description/share/dreamobot_description/urdf/dreambot.urdf.xacro (robot description, xacro)
@@ -15,4 +15,10 @@
       </geometry>
     </visual>
+    <collision>
+      <origin rpy="0 0 0" xyz="0 0 0"/>
+      <geometry>
+        <mesh filename="package://dreamobot_description/meshes/Circular_base.stl" scale="0.01 0.01 0.01"/>
+      </geometry>
+    </collision>
   </link>
   <!-- Fixed Joint: world -> base_link -->
@@ -41,5 +47,5 @@
   <link name="Arm_1" type="revolute">
     <visual>
-      <origin rpy= "0  1 4.7124" xyz="0 0 0"/>
+      <origin rpy="0 1 4.7124" xyz="0 0 0"/>
       <geometry>
         <mesh filename="package://dreamobot_description/meshes/Arm1.stl" scale="0.01 0.01 0.01"/>
@@ -47,9 +53,9 @@
     </visual>
   </link>
-  <joint name="joint_3" type='revolute'>
+  <joint name="joint_3" type="revolute">
     <parent link="base_plate"/>
     <child link="Arm_1"/>
     <axis xyz="1 0 0"/>
-    <origin rpy="0 0 0" xyz="0  0 0.4"/>
+    <origin rpy="0 0 0" xyz="0 0 0.4"/>
     <limit lower="${-PI/2}" upper="${PI/2}" effort="${effort}" velocity="${velocity}"/>
   </joint>
@@ -61,6 +67,6 @@
       </geometry>
     </visual>
-</link>
-  <joint name="joint_4" type='revolute'>
+  </link>
+  <joint name="joint_4" type="revolute">
     <parent link="Arm_1"/>
     <child link="Arm_2"/>
@@ -77,5 +83,5 @@
     </visual>
   </link>
-  <joint name="joint_5" type='revolute'>
+  <joint name="joint_5" type="revolute">
     <parent link="Arm_2"/>
     <child link="Arm_3"/>
@@ -84,36 +90,38 @@
     <limit lower="${-PI/2}" upper="${PI/2}" effort="${effort}" velocity="${velocity}"/>
   </joint>
-  <link name="Gripper_Base" type="revolute">
-    <visual>
-      <origin rpy="0 3.1416  1.5708" xyz="0.2 0.01 0"/>
+  <!-- ================== GRIPPER BASE ================== -->
+  <link name="Gripper_Base">
+    <visual>
+      <origin rpy="0 3.1416 1.5708" xyz="0.2 0.01 0"/>
       <geometry>
         <mesh filename="package://dreamobot_description/meshes/Gripper Base.stl" scale="0.01 0.01 0.01"/>
       </geometry>
     </visual>
-</link>
-<joint name="joint_6 " type="revolute">
-  <parent link="Arm_3"/>
-  <child link="Gripper_Base"/>
-  <axis xyz="1 0 0"/>
-  <origin rpy="0 0 0" xyz="0 0.25 0"/>
-  <limit lower="${-PI/2}" upper="${PI/2}" effort="${effort}" velocity="${velocity}"/>"
-</joint>
-<link name="Gear_Arm_1" type="revolute">
-  <visual>
-    <origin rpy="0 0 0" xyz="0 0 0"/>
-    <geometry>
-      <mesh filename="package://dreamobot_description/meshes/Gear Arm1.stl" scale="0.01 0.01 0.01"/>
-    </geometry>
-  </visual>
-</link>
-<link name="GearArm_2" type="revolute">
-  <visual>
-    <origin rpy="0 0 0" xyz="0 0 0"/>
-    <geometry>
-      <mesh filename="package://dreamobot_description/meshes/Gear Arm2.stl" scale="0.01 0.01 0.01"/>
-    </geometry>
-  </visual>
-</link>
-<!-- ================== LEFT GEAR ================== -->
+  </link>
+  <joint name="joint_6" type="revolute">
+    <parent link="Arm_3"/>
+    <child link="Gripper_Base"/>
+    <axis xyz="1 0 0"/>
+    <origin rpy="0 0 0" xyz="0 0.25 0"/>
+    <limit lower="${-PI/2}" upper="${PI/2}" effort="${effort}" velocity="${velocity}"/>
+  </joint>
+  <!-- ================== GEARS ================== -->
+  <link name="Gear_Arm_1">
+    <visual>
+      <origin rpy="0 0 0" xyz="0 0 0"/>
+      <geometry>
+        <mesh filename="package://dreamobot_description/meshes/Gear Arm1.stl" scale="0.01 0.01 0.01"/>
+      </geometry>
+    </visual>
+  </link>
+  <link name="Gear_Arm_2">
+    <visual>
+      <origin rpy="0 0 0" xyz="0 0 0"/>
+      <geometry>
+        <mesh filename="package://dreamobot_description/meshes/Gear Arm2.stl" scale="0.01 0.01 0.01"/>
+      </geometry>
+    </visual>
+  </link>
+  <!-- ================== LEFT GEAR ================== -->
 <joint name="joint_7" type="revolute">
   <parent link="Gripper_Base"/>
@@ -121,5 +129,5 @@
   <axis xyz="0 0 1"/>
   <origin rpy="0 0 0.7854" xyz="0.271 0.305 0.100"/>
-  <mimic joint="joint_9" multiplier="-1.0"/>
+  <mimic joint="joint_9" multiplier="1.0"/>
   <limit lower="-1.5708" upper="1.5708" effort="${effort}" velocity="${velocity}"/>
 </joint>
@@ -167,73 +175,67 @@
 </joint>
 <!-- ================== SUPPORT LINKS ================== -->
-  <!-- Grip Link 1 -->
-  <link name="Grip_link1">
-    <visual>
-      <origin rpy="0 0 3.141593" xyz="0 0 0.1"/>
-      <geometry>
-        <mesh filename="package://dreamobot_description/meshes/Gripper_Link.stl" scale="0.01 0.01 0.01"/>
-      </geometry>
-    </visual>
-  </link>
-  <joint name="joint_11" type="revolute">
-    <parent link="Gripper_Base"/>
-    <child link="Grip_link1"/>
-    <axis xyz="0 0 1"/>
-    <origin rpy="0 0 0.7854" xyz="0.192 0.514 0"/>
-    <mimic joint="joint_9" multiplier="-1.0"/>
-    <limit lower="-1.5708" upper="1.5708" effort="1.0" velocity="1.0"/>
-  </joint>
-  <!-- Grip Link 2 -->
-  <link name="Grip_link2">
-    <visual>
-      <origin rpy="0 0 3.141593" xyz="0 0 -0.05"/>
-      <geometry>
-        <mesh filename="package://dreamobot_description/meshes/Gripper_Link.stl" scale="0.01 0.01 0.01"/>
-      </geometry>
-    </visual>
-  </link>
-  <joint name="joint_12" type="revolute">
-    <parent link="Gripper_Base"/>
-    <child link="Grip_link2"/>
-    <axis xyz="0 0 1"/>
-    <origin rpy="0 0 0.7854" xyz="0.192 0.514 0"/>
-    <mimic joint="joint_9" multiplier="-1.0"/>
-    <limit lower="-1.5708" upper="1.5708" effort="1.0" velocity="1.0"/>
-  </joint>
-  <!-- Grip Link 3 -->
-  <link name="Grip_link3">
-    <visual>
-      <origin rpy="0 0 0" xyz="0 0 0.05"/>
-      <geometry>
-        <mesh filename="package://dreamobot_description/meshes/Gripper_Link.stl" scale="0.01 0.01 0.01"/>
-      </geometry>
-    </visual>
-  </link>
-  <joint name="joint_13" type="revolute">
-    <parent link="Gripper_Base"/>
-    <child link="Grip_link3"/>
-    <axis xyz="0 0 1"/>
-    <!-- mirrored position compared to Grip_link1 -->
-    <origin rpy="0 0 -0.7854" xyz="-0.192 0.514 0"/>
-    <mimic joint="joint_9" multiplier="-1.0"/>
-    <limit lower="-1.5708" upper="1.5708" effort="1.0" velocity="1.0"/>
-  </joint>
-  <!-- Grip Link 4 -->
-  <link name="Grip_link4">
-    <visual>
-      <origin rpy="0 0 0" xyz="0 0 -0.05"/>
-      <geometry>
-        <mesh filename="package://dreamobot_description/meshes/Gripper_Link.stl" scale="0.01 0.01 0.01"/>
-      </geometry>
-    </visual>
-  </link>
-  <joint name="joint_14" type="revolute">
-    <parent link="Gripper_Base"/>
-    <child link="Grip_link4"/>
-    <axis xyz="0 0 1"/>
-    <!-- mirrored position compared to Grip_link2 -->
-    <origin rpy="0 0 -0.7854" xyz="-0.192 0.514 0"/>
-    <mimic joint="joint_9" multiplier="-1.0"/>
-    <limit lower="-1.5708" upper="1.5708" effort="1.0" velocity="1.0"/>
-  </joint>
+<link name="Grip_link1">
+  <visual>
+    <origin rpy="0 0 3.141593" xyz="0 0 0.1"/>
+    <geometry>
+      <mesh filename="package://dreamobot_description/meshes/Gripper_Link.stl" scale="0.01 0.01 0.01"/>
+    </geometry>
+  </visual>
+</link>
+<joint name="joint_11" type="revolute">
+  <parent link="Gripper_Base"/>
+  <child link="Grip_link1"/>
+  <axis xyz="0 0 1"/>
+  <origin rpy="0 0 0.7854" xyz="0.192 0.514 0"/>
+  <mimic joint="joint_9" multiplier="-1.0"/>
+  <limit lower="-1.5708" upper="1.5708" effort="1.0" velocity="1.0"/>
+</joint>
+<link name="Grip_link2">
+  <visual>
+    <origin rpy="0 0 3.141593" xyz="0 0 -0.05"/>
+    <geometry>
+      <mesh filename="package://dreamobot_description/meshes/Gripper_Link.stl" scale="0.01 0.01 0.01"/>
+    </geometry>
+  </visual>
+</link>
+<joint name="joint_12" type="revolute">
+  <parent link="Gripper_Base"/>
+  <child link="Grip_link2"/>
+  <axis xyz="0 0 1"/>
+  <origin rpy="0 0 0.7854" xyz="0.192 0.514 0"/>
+  <mimic joint="joint_9" multiplier="-1.0"/>
+  <limit lower="-1.5708" upper="1.5708" effort="1.0" velocity="1.0"/>
+</joint>
+<link name="Grip_link3">
+  <visual>
+    <origin rpy="0 0 0" xyz="0 0 0.05"/>
+    <geometry>
+      <mesh filename="package://dreamobot_description/meshes/Gripper_Link.stl" scale="0.01 0.01 0.01"/>
+    </geometry>
+  </visual>
+</link>
+<joint name="joint_13" type="revolute">
+  <parent link="Gripper_Base"/>
+  <child link="Grip_link3"/>
+  <axis xyz="0 0 1"/>
+  <origin rpy="0 0 0" xyz="-1 0.5 0"/>
+  <mimic joint="joint_9" multiplier="-1.0"/>
+  <limit lower="-1.5708" upper="1.5708" effort="1.0" velocity="1.0"/>
+</joint>
+<link name="Grip_link4">
+  <visual>
+    <origin rpy="0 0 0" xyz="0 0 -0.05"/>
+    <geometry>
+      <mesh filename="package://dreamobot_description/meshes/Gripper_Link.stl" scale="0.01 0.01 0.01"/>
+    </geometry>
+  </visual>
+</link>
+<joint name="joint_14" type="revolute">
+  <parent link="Gripper_Base"/>
+  <child link="Grip_link4"/>
+  <axis xyz="0 0 1"/>
+  <origin rpy="0 0 0" xyz="-1 0.5 0"/>
+  <mimic joint="joint_9" multiplier="-1.0"/>
+  <limit lower="-1.5708" upper="1.5708" effort="1.0" velocity="1.0"/>
+</joint>
 </robot>
